Commit message: modify link2 flying_arm_2

File: robots/borinot_flying_arm_2/borinot_flying_arm_2.urdf (robot description, URDF)
Before this commit: robot borinot_flynig_arm_2, 4 links, 3 joints
Links:
- link flying_arm_2__link2: mass 0.0631438822022442 -> 0.115
Joints:
- joint flying_arm_2__j_link2_ee: origin xyz=0 -0.15 0 rpy=0 0 -1.5708 -> xyz=0 -0.130 0 rpy=0 0 -1.5708

Commit message: modify borinot_flying_arm_2 end-effector

File: robots/borinot_flying_arm_2/borinot_flying_arm_2.urdf (robot description, URDF)
Before this commit: robot borinot_flynig_arm_2, 4 links, 3 joints
Links:
- link flying_arm_2__ee: mass 0.1 -> 0.0
