Commit message: modify borinot parameters

File: robots/borinot/borinot.urdf (robot description, URDF)
Before this commit: robot borinot, 1 links, 0 joints
Links:
- link borinot__base_link: mass 2.085 -> 2.049

Commit message: feat: minor imporvements

File: robots/borinot/borinot.urdf (robot description, URDF)
Before this commit: robot borinot, 1 links, 0 joints
Links:
- added link borinot__rotor0, mass 0.005; collision cylinder length=0.005 radius=0.070; visual mesh filename=package://hidro_robots/robots/common/meshes/propeller_cw.dae scale=0.1 0.1 0.1
- added link borinot__rotor1, mass 0.005; collision cylinder length=0.005 radius=0.070; visual mesh filename=package://hidro_robots/robots/common/meshes/propeller_ccw.d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 scale=0.1 0.1 0.1
- added link borinot__rotor2, mass 0.005; collision cylinder length=0.005 radius=0.070; visual mesh filename=package://hidro_robots/robots/common/meshes/propeller_cw.dae scale=0.1 0.1 0.1
- added link borinot__rotor3, mass 0.005; collision cylinder length=0.005 radius=0.070; visual mesh filename=package://hidro_robots/robots/common/meshes/propeller_ccw.d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 scale=0.1 0.1 0.1
- added link borinot__rotor4, mass 0.005; collision cylinder length=0.005 radius=0.070; visual mesh filename=package://hidro_robots/robots/common/meshes/propeller_ccw.d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 scale=0.1 0.1 0.1
- added link borinot__rotor5, mass 0.005; collision cylinder length=0.005 radius=0.070; visual mesh filename=package://hidro_robots/robots/common/meshes/propeller_cw.dae scale=0.1 0.1 0.1
- link borinot__base_link: geometry collision box size=0.4 0.4 0.3; visual mesh filename=package://hidro_robots/robots/borinot/meshes/borinot__base_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 scale=1 1 1
Joints:
- added joint borinot__j_rotor0: type fixed, parent borinot__base_link, child borinot__rotor0, origin xyz=0.0 -0.185 0.05 rpy=0.0 0 0.0, axis 0 0 1, limit lower=-1e16 upper=1e16 effort=10 velocity=1e16
- added joint borinot__j_rotor1: type fixed, parent borinot__base_link, child borinot__rotor1, origin xyz=0.0 0.185 0.05 rpy=0.0 0 0.0, axis 0 0 1, limit lower=-1e16 upper=1e16 effort=10 velocity=1e16
- added joint borinot__j_rotor2: type fixed, parent borinot__base_link, child borinot__rotor2, origin xyz=0.1602146997 0.0925 0.05 rpy=0.0 0 0.0, axis 0 0 1, limit lower=-1e16 upper=1e16 effort=10 velocity=1e16
- added joint borinot__j_rotor3: type fixed, parent borinot__base_link, child borinot__rotor3, origin xyz=-0.1602146997 -0.0925 0.05 rpy=0.0 0 0.0, axis 0 0 1, limit lower=-1e16 upper=1e16 effort=10 velocity=1e16
- added joint borinot__j_rotor4: type fixed, parent borinot__base_link, child borinot__rotor4, origin xyz=0.1602146997 -0.0925 0.05 rpy=0.0 0 0.0, axis 0 0 1, limit lower=-1e16 upper=1e16 effort=10 velocity=1e16
- added joint borinot__j_rotor5: type fixed, parent borinot__base_link, child borinot__rotor5, origin xyz=-0.1602146997 0.0925 0.05 rpy=0.0 0 0.0, axis 0 0 1, limit lower=-1e16 upper=1e16 effort=10 velocity=1e16

File: robots/borinot/xacro/definition.urdf.xacro (robot description, xacro)
@@ -5,18 +5,33 @@
   <xacro:include
     filename="$(find hidro_robots)/robots/common/xacro/sensors.xacro" />
-  <xacro:macro name="borinot_platform" params="simulation">
+  <xacro:macro name="borinot_platform" params="robot_name simulation has_arm">
     <xacro:property name="platform_name" value="borinot" />
     <!-- platform -->
-    <xacro:platform
-      platform_name="${platform_name}"
-      mass="2.049"
-      cog_x="0.0"
-      cog_y="0.0"
-      cog_z="0.0341"
-      i_xx="0.017598"
-      i_yy="0.017957"
-      i_zz="0.029599"
-      mesh="package://hidro_robots/robots/borinot/meshes/borinot__base_link.dae"
-    />
+    <xacro:unless value="${has_arm}">
+      <xacro:platform
+        platform_name="${platform_name}"
+        mass="2.049"
+        cog_x="0.0"
+        cog_y="0.0"
+        cog_z="0.0341"
+        i_xx="0.017598"
+        i_yy="0.017957"
+        i_zz="0.029599"
+        mesh="package://hidro_robots/robots/borinot/meshes/borinot__base_link.dae"
+      />
+    </xacro:unless>
+    <xacro:if value="${has_arm}">
+      <xacro:platform
+        platform_name="${platform_name}"
+        mass="2.647"
+        cog_x="0.0"
+        cog_y="0.00244"
+        cog_z="0.0202"
+        i_xx="0.027246422051605018"
+        i_yy="0.026854677520396303"
+        i_zz="0.039807168462897885"
+        mesh="package://hidro_robots/robots/borinot/meshes/borinot__base_link__arm.dae"
+      />
+    </xacro:if>
     <!-- rotors -->
     <xacro:rotor
@@ -82,4 +97,5 @@
     <xacro:if value="${simulation}">
       <xacro:px4_plugins
+        robot_name="${robot_name}"
         platform_name="${platform_name}"
       />

File: robots/borinot/xacro/description.urdf.xacro (robot description, xacro)
@@ -12,5 +12,7 @@
   <xacro:property name="simulation" value="$(arg simulation)" />
   <xacro:borinot_platform
+    robot_name="borinot"
     simulation="${simulation}"
+    has_arm="false"
   />
 </robot>

File: robots/borinot_flying_arm_2/borinot_flying_arm_2.urdf (robot description, URDF)
Before this commit: robot borinot_flynig_arm_2, 4 links, 3 joints
Links:
- added link borinot__rotor0, mass 0.005; collision cylinder length=0.005 radius=0.070; visual mesh filename=package://hidro_robots/robots/common/meshes/propeller_cw.dae scale=0.1 0.1 0.1
- added link borinot__rotor1, mass 0.005; collision cylinder length=0.005 radius=0.070; visual mesh filename=package://hidro_robots/robots/common/meshes/propeller_ccw.d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 scale=0.1 0.1 0.1
- added link borinot__rotor2, mass 0.005; collision cylinder length=0.005 radius=0.070; visual mesh filename=package://hidro_robots/robots/common/meshes/propeller_cw.dae scale=0.1 0.1 0.1
- added link borinot__rotor3, mass 0.005; collision cylinder length=0.005 radius=0.070; visual mesh filename=package://hidro_robots/robots/common/meshes/propeller_ccw.d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 scale=0.1 0.1 0.1
- added link borinot__rotor4, mass 0.005; collision cylinder length=0.005 radius=0.070; visual mesh filename=package://hidro_robots/robots/common/meshes/propeller_ccw.d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 scale=0.1 0.1 0.1
- added link borinot__rotor5, mass 0.005; collision cylinder length=0.005 radius=0.070; visual mesh filename=package://hidro_robots/robots/common/meshes/propeller_cw.dae scale=0.1 0.1 0.1
- link borinot__base_link: geometry collision box size=0.4 0.4 0.3; visual mesh filename=package://hidro_robots/robots/borinot/meshes/borinot__base_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 scale=1 1 1
- link flying_arm_2__link1: geometry visual mesh filename=package://hidro_robots/robots/borinot_flying_arm_2/meshes/f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
- link flying_arm_2__link2: geometry visual mesh filename=package://hidro_robots/robots/borinot_flying_arm_2/meshes/f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
Joints:
- added joint borinot__j_rotor0: type fixed, parent borinot__base_link, child borinot__rotor0, origin xyz=0.0 -0.185 0.05 rpy=0.0 0 0.0, axis 0 0 1, limit lower=-1e16 upper=1e16 effort=10 velocity=1e16
- added joint borinot__j_rotor1: type fixed, parent borinot__base_link, child borinot__rotor1, origin xyz=0.0 0.185 0.05 rpy=0.0 0 0.0, axis 0 0 1, limit lower=-1e16 upper=1e16 effort=10 velocity=1e16
- added joint borinot__j_rotor2: type fixed, parent borinot__base_link, child borinot__rotor2, origin xyz=0.1602146997 0.0925 0.05 rpy=0.0 0 0.0, axis 0 0 1, limit lower=-1e16 upper=1e16 effort=10 velocity=1e16
- added joint borinot__j_rotor3: type fixed, parent borinot__base_link, child borinot__rotor3, origin xyz=-0.1602146997 -0.0925 0.05 rpy=0.0 0 0.0, axis 0 0 1, limit lower=-1e16 upper=1e16 effort=10 velocity=1e16
- added joint borinot__j_rotor4: type fixed, parent borinot__base_link, child borinot__rotor4, origin xyz=0.1602146997 -0.0925 0.05 rpy=0.0 0 0.0, axis 0 0 1, limit lower=-1e16 upper=1e16 effort=10 velocity=1e16
- added joint borinot__j_rotor5: type fixed, parent borinot__base_link, child borinot__rotor5, origin xyz=-0.1602146997 0.0925 0.05 rpy=0.0 0 0.0, axis 0 0 1, limit lower=-1e16 upper=1e16 effort=10 velocity=1e16
- joint flying_arm_2__j_link1_link2: limit lower=-1.6707963267948966 upper=1.6707963267948966 effort=2.5 velocity=10000 -> lower=-3.1 upper=3.1 effort=2.5 velocity=10000

File: robots/borinot_flying_arm_2/xacro/description.urdf.xacro (robot description, xacro)
@@ -1,3 +1,3 @@
-<robot name="borinot" xmlns:xacro="http://www.ros.org/wiki/xacro">
+<robot name="borinot_flying_arm_2" xmlns:xacro="http://www.ros.org/wiki/xacro">
   <!-- macro includes -->
   <xacro:include
@@ -10,5 +10,7 @@
   <xacro:property name="simulation" value="$(arg simulation)" />
   <xacro:borinot_platform
+    robot_name="borinot_flying_arm_2"
     simulation="${simulation}"
+    has_arm="true"
   />
   <xacro:flying_arm_2
@@ -16,3 +18,14 @@
     base_link_name="borinot__base_link"
   />
+  <gazebo>
+    <plugin name='external_force_plugin' filename='libeagle_gazebo_force_plugin.so'>
+      <namespace>borinot_flying_arm_2</namespace>
+      <trajectoryName>aasquare.yaml</trajectoryName>
+      <linkName>borinot__base_link</linkName>
+      <direction>1 0 0</direction>
+      <instant>1.0</instant>
+      <magnitude>30.0</magnitude>
+      <duration>1.0</duration>
+    </plugin>
+  </gazebo>
 </robot>

File: robots/common/xacro/multicopter.xacro (robot description, xacro)
@@ -79,5 +79,5 @@
           <timeConstantDown>0.005</timeConstantDown>
           <maxRotVelocity>2236</maxRotVelocity>
-          <motorConstant>4.511e-06</motorConstant>
+          <motorConstant>3.847e-6</motorConstant>
           <momentConstant>0.06</momentConstant>
           <commandSubTopic>/gazebo/command/motor_speed</commandSubTopic>

File: robots/common/xacro/sensors.xacro (robot description, xacro)
@@ -15,4 +15,5 @@
     </joint>
     <gazebo>
+      <!-- Ideal IMU config -->
       <plugin name='imu_plugin' filename='libgazebo_imu_plugin.so'>
         <robotNamespace />
@@ -21,14 +22,30 @@
         <gyroscopeNoiseDensity>0.0</gyroscopeNoiseDensity>
         <gyroscopeRandomWalk>0.0</gyroscopeRandomWalk>
-        <gyroscopeBiasCorrelationTime>10.0</gyroscopeBiasCorrelationTime>
+        <gyroscopeBiasCorrelationTime>1000</gyroscopeBiasCorrelationTime>
         <gyroscopeTurnOnBiasSigma>0.00</gyroscopeTurnOnBiasSigma>
         <accelerometerNoiseDensity>0.0</accelerometerNoiseDensity>
         <accelerometerRandomWalk>0.0</accelerometerRandomWalk>
-        <accelerometerBiasCorrelationTime>3.0</accelerometerBiasCorrelationTime>
+        <accelerometerBiasCorrelationTime>300</accelerometerBiasCorrelationTime>
         <accelerometerTurnOnBiasSigma>0.0</accelerometerTurnOnBiasSigma>
       </plugin>
     </gazebo>
+    <!-- Noisy + bias IMU config -->
+    <!-- <gazebo>
+      <plugin name='imu_plugin' filename='libgazebo_imu_plugin.so'>
+        <robotNamespace />
+        <linkName>${platform_name}__imu</linkName>
+        <imuTopic>/imu</imuTopic>
+        <gyroscopeNoiseDensity>0.00018665</gyroscopeNoiseDensity>
+        <gyroscopeRandomWalk>3.8785e-05</gyroscopeRandomWalk>
+        <gyroscopeBiasCorrelationTime>1000.0</gyroscopeBiasCorrelationTime>
+        <gyroscopeTurnOnBiasSigma>0.0087</gyroscopeTurnOnBiasSigma>
+        <accelerometerNoiseDensity>0.00186</accelerometerNoiseDensity>
+        <accelerometerRandomWalk>0.006</accelerometerRandomWalk>
+        <accelerometerBiasCorrelationTime>300.0</accelerometerBiasCorrelationTime>
+        <accelerometerTurnOnBiasSigma>0.196</accelerometerTurnOnBiasSigma>
+      </plugin>
+    </gazebo> -->
   </xacro:macro>
-  <xacro:macro name="px4_plugins" params="platform_name">
+  <xacro:macro name="px4_plugins" params="robot_name platform_name ">
     <!-- IMU -->
     <xacro:imu
@@ -63,5 +80,15 @@
     <!-- MAGNETOMETER -->
     <gazebo>
+      <!-- Ideal Magneto config -->
       <plugin name='magnetometer_plugin' filename='libgazebo_magnetometer_plugin.so'>
+        <robotNamespace />
+        <pubRate>100</pubRate>
+        <noiseDensity>0.0</noiseDensity>
+        <randomWalk>0.0</randomWalk>
+        <biasCorrelationTime>600</biasCorrelationTime>
+        <magTopic>/mag</magTopic>
+      </plugin>
+      <!-- Noisy + bias Magneto config -->
+      <!-- <plugin name='magnetometer_plugin' filename='libgazebo_magnetometer_plugin.so'>
         <robotNamespace />
         <pubRate>100</pubRate>
@@ -70,5 +97,5 @@
         <biasCorrelationTime>600</biasCorrelationTime>
         <magTopic>/mag</magTopic>
-      </plugin>
+      </plugin> -->
     </gazebo>
     <!-- BAROMETER -->
@@ -78,4 +105,5 @@
         <pubRate>50</pubRate>
         <baroTopic>/baro</baroTopic>
+        <baroDriftPaPerSec>0</baroDriftPaPerSec>
       </plugin>
     </gazebo>

File: robots/flying_arm_2/xacro/definition.urdf.xacro (robot description, xacro)
@@ -105,9 +105,13 @@
           <joint name="flying_arm_2__j_bl_link1">
             <param name="safe_position">-1.3</param>
-            <param name="safe_torque">-0.4</param>
+            <param name="safe_torque">-0.3</param>
+            <param name="safe_pos_gain">2.0</param>
+            <param name="safe_vel_gain">0.2</param>
           </joint>
           <joint name="flying_arm_2__j_link1_link2">
             <param name="safe_position">2.8</param>
-            <param name="safe_torque">0.2</param>
+            <param name="safe_torque">0.1</param>
+            <param name="safe_pos_gain">2.0</param>
+            <param name="safe_vel_gain">0.2</param>
           </joint>
         </plugin>
