Commit message: feat: adapt descriptions for event-based simulation

File: robots/borinot/xacro/definition.urdf.xacro (robot description, xacro)
@@ -5,5 +5,5 @@
   <xacro:include
     filename="$(find hidro_robots)/robots/common/xacro/sensors.xacro" />
-  <xacro:macro name="borinot_platform" params="robot_name simulation has_arm">
+  <xacro:macro name="borinot_platform" params="robot_name simulation event_based_sim has_arm">
     <xacro:property name="platform_name" value="borinot" />
     <!-- platform -->
@@ -44,4 +44,5 @@
       direction="cw"
       simulation="${simulation}"
+      event_based_sim="${event_based_sim}"
     />
     <xacro:rotor
@@ -54,4 +55,5 @@
       direction="ccw"
       simulation="${simulation}"
+      event_based_sim="${event_based_sim}"
     />
     <xacro:rotor
@@ -64,4 +66,5 @@
       direction="cw"
       simulation="${simulation}"
+      event_based_sim="${event_based_sim}"
     />
     <xacro:rotor
@@ -74,4 +77,5 @@
       direction="ccw"
       simulation="${simulation}"
+      event_based_sim="${event_based_sim}"
     />
     <xacro:rotor
@@ -84,4 +88,5 @@
       direction="ccw"
       simulation="${simulation}"
+      event_based_sim="${event_based_sim}"
     />
     <xacro:rotor
@@ -94,86 +99,89 @@
       direction="cw"
       simulation="${simulation}"
+      event_based_sim="${event_based_sim}"
     />
     <xacro:if value="${simulation}">
-      <xacro:px4_plugins
-        robot_name="${robot_name}"
-        platform_name="${platform_name}"
-      />
-      <!-- MAVLINK -->
-      <gazebo>
-        <plugin name='mavlink_interface' filename='libgazebo_mavlink_interface.so'>
-          <robotNamespace />
-          <imuSubTopic>/imu</imuSubTopic>
-          <magSubTopic>/mag</magSubTopic>
-          <baroSubTopic>/baro</baroSubTopic>
-          <mavlink_addr>INADDR_ANY</mavlink_addr>
-          <mavlink_tcp_port>4560</mavlink_tcp_port>
-          <mavlink_udp_port>14560</mavlink_udp_port>
-          <serialEnabled>0</serialEnabled>
-          <serialDevice>/dev/ttyACM0</serialDevice>
-          <baudRate>921600</baudRate>
-          <qgc_addr>INADDR_ANY</qgc_addr>
-          <qgc_udp_port>14550</qgc_udp_port>
-          <sdk_addr>INADDR_ANY</sdk_addr>
-          <sdk_udp_port>14540</sdk_udp_port>
-          <hil_mode>0</hil_mode>
-          <hil_state_level>0</hil_state_level>
-          <send_vision_estimation>0</send_vision_estimation>
-          <send_odometry>1</send_odometry>
-          <enable_lockstep>1</enable_lockstep>
-          <use_tcp>1</use_tcp>
-          <motorSpeedCommandPubTopic>/gazebo/command/motor_speed</motorSpeedCommandPubTopic>
-          <control_channels>
-            <channel name='rotor1'>
-              <input_index>0</input_index>
-              <input_offset>0</input_offset>
-              <input_scaling>2136</input_scaling>
-              <zero_position_disarmed>0</zero_position_disarmed>
-              <zero_position_armed>100</zero_position_armed>
-              <joint_control_type>velocity</joint_control_type>
-            </channel>
-            <channel name='rotor2'>
-              <input_index>1</input_index>
-              <input_offset>0</input_offset>
-              <input_scaling>2136</input_scaling>
-              <zero_position_disarmed>0</zero_position_disarmed>
-              <zero_position_armed>100</zero_position_armed>
-              <joint_control_type>velocity</joint_control_type>
-            </channel>
-            <channel name='rotor3'>
-              <input_index>2</input_index>
-              <input_offset>0</input_offset>
-              <input_scaling>2136</input_scaling>
-              <zero_position_disarmed>0</zero_position_disarmed>
-              <zero_position_armed>100</zero_position_armed>
-              <joint_control_type>velocity</joint_control_type>
-            </channel>
-            <channel name='rotor4'>
-              <input_index>3</input_index>
-              <input_offset>0</input_offset>
-              <input_scaling>2136</input_scaling>
-              <zero_position_disarmed>0</zero_position_disarmed>
-              <zero_position_armed>100</zero_position_armed>
-              <joint_control_type>velocity</joint_control_type>
-            </channel>
-            <channel name='rotor5'>
-              <input_index>4</input_index>
-              <input_offset>0</input_offset>
-              <input_scaling>2136</input_scaling>
-              <zero_position_disarmed>0</zero_position_disarmed>
-              <zero_position_armed>100</zero_position_armed>
-              <joint_control_type>velocity</joint_control_type>
-            </channel>
-            <channel name='rotor6'>
-              <input_index>5</input_index>
-              <input_offset>0</input_offset>
-              <input_scaling>2136</input_scaling>
-              <zero_position_disarmed>0</zero_position_disarmed>
-              <zero_position_armed>100</zero_position_armed>
-              <joint_control_type>velocity</joint_control_type>
-            </channel>
-          </control_channels>
-        </plugin>
-      </gazebo>
+      <xacro:unless value="${event_based_sim}">
+        <xacro:px4_plugins
+          robot_name="${robot_name}"
+          platform_name="${platform_name}"
+        />
+        <!-- MAVLINK -->
+        <gazebo>
+          <plugin name='mavlink_interface' filename='libgazebo_mavlink_interface.so'>
+            <robotNamespace />
+            <imuSubTopic>/imu</imuSubTopic>
+            <magSubTopic>/mag</magSubTopic>
+            <baroSubTopic>/baro</baroSubTopic>
+            <mavlink_addr>INADDR_ANY</mavlink_addr>
+            <mavlink_tcp_port>4560</mavlink_tcp_port>
+            <mavlink_udp_port>14560</mavlink_udp_port>
+            <serialEnabled>0</serialEnabled>
+            <serialDevice>/dev/ttyACM0</serialDevice>
+            <baudRate>921600</baudRate>
+            <qgc_addr>INADDR_ANY</qgc_addr>
+            <qgc_udp_port>14550</qgc_udp_port>
+            <sdk_addr>INADDR_ANY</sdk_addr>
+            <sdk_udp_port>14540</sdk_udp_port>
+            <hil_mode>0</hil_mode>
+            <hil_state_level>0</hil_state_level>
+            <send_vision_estimation>0</send_vision_estimation>
+            <send_odometry>1</send_odometry>
+            <enable_lockstep>1</enable_lockstep>
+            <use_tcp>1</use_tcp>
+            <motorSpeedCommandPubTopic>/gazebo/command/motor_speed</motorSpeedCommandPubTopic>
+            <control_channels>
+              <channel name='rotor1'>
+                <input_index>0</input_index>
+                <input_offset>0</input_offset>
+                <input_scaling>2136</input_scaling>
+                <zero_position_disarmed>0</zero_position_disarmed>
+                <zero_position_armed>100</zero_position_armed>
+                <joint_control_type>velocity</joint_control_type>
+              </channel>
+              <channel name='rotor2'>
+                <input_index>1</input_index>
+                <input_offset>0</input_offset>
+                <input_scaling>2136</input_scaling>
+                <zero_position_disarmed>0</zero_position_disarmed>
+                <zero_position_armed>100</zero_position_armed>
+                <joint_control_type>velocity</joint_control_type>
+              </channel>
+              <channel name='rotor3'>
+                <input_index>2</input_index>
+                <input_offset>0</input_offset>
+                <input_scaling>2136</input_scaling>
+                <zero_position_disarmed>0</zero_position_disarmed>
+                <zero_position_armed>100</zero_position_armed>
+                <joint_control_type>velocity</joint_control_type>
+              </channel>
+              <channel name='rotor4'>
+                <input_index>3</input_index>
+                <input_offset>0</input_offset>
+                <input_scaling>2136</input_scaling>
+                <zero_position_disarmed>0</zero_position_disarmed>
+                <zero_position_armed>100</zero_position_armed>
+                <joint_control_type>velocity</joint_control_type>
+              </channel>
+              <channel name='rotor5'>
+                <input_index>4</input_index>
+                <input_offset>0</input_offset>
+                <input_scaling>2136</input_scaling>
+                <zero_position_disarmed>0</zero_position_disarmed>
+                <zero_position_armed>100</zero_position_armed>
+                <joint_control_type>velocity</joint_control_type>
+              </channel>
+              <channel name='rotor6'>
+                <input_index>5</input_index>
+                <input_offset>0</input_offset>
+                <input_scaling>2136</input_scaling>
+                <zero_position_disarmed>0</zero_position_disarmed>
+                <zero_position_armed>100</zero_position_armed>
+                <joint_control_type>velocity</joint_control_type>
+              </channel>
+            </control_channels>
+          </plugin>
+        </gazebo>
+      </xacro:unless>
     </xacro:if>
   </xacro:macro>

File: robots/borinot/xacro/description.urdf.xacro (robot description, xacro)
@@ -9,10 +9,61 @@
   <!-- arguments -->
   <xacro:arg name="simulation" default="true" />
+  <xacro:arg name="event_based_sim" default="false" />
   <!-- properties -->
   <xacro:property name="simulation" value="$(arg simulation)" />
+  <xacro:property name="event_based_sim" value="$(arg event_based_sim)" />
   <xacro:borinot_platform
     robot_name="borinot"
     simulation="${simulation}"
+    event_based_sim="${event_based_sim}"
     has_arm="false"
   />
+  <xacro:if value="${simulation}">
+    <xacro:if value="${event_based_sim}">
+      <gazebo>
+        <plugin name='eagle_gazebo_event_base_sim_plugin'
+          filename='libeagle_gazebo_event_based_sim_plugin.so'>
+          <simulationRate>2000</simulationRate>
+          <actuationRate>500</actuationRate>
+          <uamStateTopic>/borinot/uam_state</uamStateTopic>
+          <uamControlTopic>/borinot/uam_control</uamControlTopic>
+          <platform_params>
+            <baselinkName>borinot__base_link</baselinkName>
+            <thrustToTorqueRatio>0.01393568</thrustToTorqueRatio>
+            <rotor_params>
+              <number>0</number>
+              <linkName>borinot__rotor0</linkName>
+              <turningDirection>-1</turningDirection>
+            </rotor_params>
+            <rotor_params>
+              <number>1</number>
+              <linkName>borinot__rotor1</linkName>
+              <turningDirection>1</turningDirection>
+            </rotor_params>
+            <rotor_params>
+              <number>2</number>
+              <linkName>borinot__rotor2</linkName>
+              <turningDirection>-1</turningDirection>
+            </rotor_params>
+            <rotor_params>
+              <number>3</number>
+              <linkName>borinot__rotor3</linkName>
+              <turningDirection>1</turningDirection>
+            </rotor_params>
+            <rotor_params>
+              <number>4</number>
+              <linkName>borinot__rotor4</linkName>
+              <turningDirection>1</turningDirection>
+            </rotor_params>
+            <rotor_params>
+              <number>5</number>
+              <linkName>borinot__rotor5</linkName>
+              <turningDirection>-1</turningDirection>
+            </rotor_params>
+          </platform_params>
+          <!-- here add the arm -->
+        </plugin>
+      </gazebo>
+    </xacro:if>
+  </xacro:if>
 </robot>

File: robots/borinot_flying_arm_2/xacro/description.urdf.xacro (robot description, xacro)
@@ -7,18 +7,23 @@
   <!-- arguments -->
   <xacro:arg name="simulation" default="true" />
+  <xacro:arg name="event_based_sim" default="false" />
   <!-- properties -->
   <xacro:property name="simulation" value="$(arg simulation)" />
+  <xacro:property name="event_based_sim" value="$(arg event_based_sim)" />
+  <xacro:property name="robot_name" value="borinot_flying_arm_2" />
   <xacro:borinot_platform
-    robot_name="borinot_flying_arm_2"
+    robot_name="${robot_name}"
     simulation="${simulation}"
     has_arm="true"
+    event_based_sim="${event_based_sim}"
   />
   <xacro:flying_arm_2
     simulation="${simulation}"
     base_link_name="borinot__base_link"
+    event_based_sim="${event_based_sim}"
   />
   <gazebo>
     <plugin name='external_force_plugin' filename='libeagle_gazebo_force_plugin.so'>
-      <namespace>borinot_flying_arm_2</namespace>
+      <namespace>${robot_name}</namespace>
       <trajectoryName>aasquare.yaml</trajectoryName>
       <linkName>borinot__base_link</linkName>
@@ -29,3 +34,60 @@
     </plugin>
   </gazebo>
+  <xacro:if value="${simulation}">
+    <xacro:if value="${event_based_sim}">
+      <gazebo>
+        <plugin name='eagle_gazebo_event_base_sim_plugin'
+          filename='libeagle_gazebo_event_based_sim_plugin.so'>
+          <simulationRate>2000</simulationRate>
+          <actuationRate>500</actuationRate>
+          <uamStateTopic>/${robot_name}/uam_state</uamStateTopic>
+          <uamControlTopic>/${robot_name}/uam_control</uamControlTopic>
+          <platform_params>
+            <baselinkName>borinot__base_link</baselinkName>
+            <thrustToTorqueRatio>0.01393568</thrustToTorqueRatio>
+            <rotor_params>
+              <number>0</number>
+              <linkName>borinot__rotor0</linkName>
+              <turningDirection>-1</turningDirection>
+            </rotor_params>
+            <rotor_params>
+              <number>1</number>
+              <linkName>borinot__rotor1</linkName>
+              <turningDirection>1</turningDirection>
+            </rotor_params>
+            <rotor_params>
+              <number>2</number>
+              <linkName>borinot__rotor2</linkName>
+              <turningDirection>-1</turningDirection>
+            </rotor_params>
+            <rotor_params>
+              <number>3</number>
+              <linkName>borinot__rotor3</linkName>
+              <turningDirection>1</turningDirection>
+            </rotor_params>
+            <rotor_params>
+              <number>4</number>
+              <linkName>borinot__rotor4</linkName>
+              <turningDirection>1</turningDirection>
+            </rotor_params>
+            <rotor_params>
+              <number>5</number>
+              <linkName>borinot__rotor5</linkName>
+              <turningDirection>-1</turningDirection>
+            </rotor_params>
+          </platform_params>
+          <arm_params>
+            <joint_params>
+              <number>0</number>
+              <jointName>flying_arm_2__j_bl_link1</jointName>
+            </joint_params>
+            <joint_params>
+              <number>1</number>
+              <jointName>flying_arm_2__j_link1_link2</jointName>
+            </joint_params>
+          </arm_params>
+        </plugin>
+      </gazebo>
+    </xacro:if>
+  </xacro:if>
 </robot>

File: robots/common/xacro/multicopter.xacro (robot description, xacro)
@@ -27,5 +27,5 @@
   </xacro:macro>
   <xacro:macro name="rotor"
-    params="platform_name rotor_number parent_link x y z direction simulation">
+    params="platform_name rotor_number parent_link x y z direction simulation event_based_sim">
     <xacro:property name="link_name" value="${platform_name}__rotor${rotor_number}" />
     <xacro:property name="joint_name" value="${platform_name}__j_rotor${rotor_number}" />
@@ -70,23 +70,25 @@
     </joint>
     <xacro:if value="${simulation}">
-      <gazebo>
-        <plugin name='${joint_name}_plugin' filename='libgazebo_motor_model.so'>
-          <robotNamespace></robotNamespace>
-          <jointName>${joint_name}</jointName>
-          <linkName>${link_name}</linkName>
-          <turningDirection>${direction_rotation}</turningDirection>
-          <timeConstantUp>0.005</timeConstantUp>
-          <timeConstantDown>0.005</timeConstantDown>
-          <maxRotVelocity>2236</maxRotVelocity>
-          <motorConstant>3.847e-6</motorConstant>
-          <momentConstant>0.06</momentConstant>
-          <commandSubTopic>/gazebo/command/motor_speed</commandSubTopic>
-          <motorNumber>${rotor_number}</motorNumber>
-          <rotorDragCoefficient>0.000175</rotorDragCoefficient>
-          <rollingMomentCoefficient>1e-06</rollingMomentCoefficient>
-          <motorSpeedPubTopic>/motor_speed/${rotor_number}</motorSpeedPubTopic>
-          <rotorVelocitySlowdownSim>10</rotorVelocitySlowdownSim>
-        </plugin>
-      </gazebo>
+      <xacro:unless value="${event_based_sim}">
+        <gazebo>
+          <plugin name='${joint_name}_plugin' filename='libgazebo_motor_model.so'>
+            <robotNamespace></robotNamespace>
+            <jointName>${joint_name}</jointName>
+            <linkName>${link_name}</linkName>
+            <turningDirection>${direction_rotation}</turningDirection>
+            <timeConstantUp>0.005</timeConstantUp>
+            <timeConstantDown>0.005</timeConstantDown>
+            <maxRotVelocity>2236</maxRotVelocity>
+            <motorConstant>3.847e-6</motorConstant>
+            <momentConstant>0.06</momentConstant>
+            <commandSubTopic>/gazebo/command/motor_speed</commandSubTopic>
+            <motorNumber>${rotor_number}</motorNumber>
+            <rotorDragCoefficient>0.000175</rotorDragCoefficient>
+            <rollingMomentCoefficient>1e-06</rollingMomentCoefficient>
+            <motorSpeedPubTopic>/motor_speed/${rotor_number}</motorSpeedPubTopic>
+            <rotorVelocitySlowdownSim>10</rotorVelocitySlowdownSim>
+          </plugin>
+        </gazebo>
+      </xacro:unless>
     </xacro:if>
   </xacro:macro>

File: robots/flying_arm_2/xacro/definition.urdf.xacro (robot description, xacro)
@@ -1,4 +1,4 @@
 <robot xmlns:xacro="http://www.ros.org/wiki/xacro">
-  <xacro:macro name="flying_arm_2" params="simulation base_link_name">
+  <xacro:macro name="flying_arm_2" params="simulation event_based_sim base_link_name">
     <xacro:property name="platform_name" value="borinot" />
     <xacro:if value="${base_link_name==''}">
@@ -101,20 +101,22 @@
     </joint>
     <xacro:if value="${simulation}">
-      <gazebo>
-        <plugin name="odri_gazebo" filename="libodri_gazebo_plugin.so">
-          <joint name="flying_arm_2__j_bl_link1">
-            <param name="safe_position">-1.3</param>
-            <param name="safe_torque">-0.3</param>
-            <param name="safe_pos_gain">2.0</param>
-            <param name="safe_vel_gain">0.2</param>
-          </joint>
-          <joint name="flying_arm_2__j_link1_link2">
-            <param name="safe_position">2.8</param>
-            <param name="safe_torque">0.1</param>
-            <param name="safe_pos_gain">2.0</param>
-            <param name="safe_vel_gain">0.2</param>
-          </joint>
-        </plugin>
-      </gazebo>
+      <xacro:unless value="${event_based_sim}">
+        <gazebo>
+          <plugin name="odri_gazebo" filename="libodri_gazebo_plugin.so">
+            <joint name="flying_arm_2__j_bl_link1">
+              <param name="safe_position">-1.3</param>
+              <param name="safe_torque">-0.3</param>
+              <param name="safe_pos_gain">2.0</param>
+              <param name="safe_vel_gain">0.2</param>
+            </joint>
+            <joint name="flying_arm_2__j_link1_link2">
+              <param name="safe_position">2.8</param>
+              <param name="safe_torque">0.1</param>
+              <param name="safe_pos_gain">2.0</param>
+              <param name="safe_vel_gain">0.2</param>
+            </joint>
+          </plugin>
+        </gazebo>
+      </xacro:unless>
     </xacro:if>
   </xacro:macro>
